File: ph_air_shower_controller_hw/ph_air_shower_controller_hw.sch (KiCad schematic (older format))
At the start: 176 parts, among them J1 Conn_01x02, J2 Conn_01x02, J3 Conn_01x04, J4 Conn_01x06, J5 Conn_01x04, J6 Conn_01x10, J7 Conn_01x06, J8 Conn_01x06, P1 USB_OTG, Q1 C1815, Q2 LN2302, Q3 LN2302, Q4 C1815, Q5 LN2302, Q6 LN2302, Q7 C1815, Q8 LN2302, Q9 LN2302, SW1 RESET, SW2 SW_Push, SW3 SW_Push, SW4 SW_Push, SW5 SW_Push, U1 W25Q80BV, U10 PC817, U11 ULN2803A, U12 PC817, U13 PC817, U14 PC817, U15 PC817, U16 DS18B20, U2 MC34063, U3 MAX485, U4 ASM1117, U5 SM5852, U6 SM5852, U7 STM32F103RD, U8 74HC245, U9 PC817, Y1 8Mhz, Y2 32768Khz

Commit message: Update
Parts:
- removed C15, C29: 100nF, Capacitor_SMD:C_0805_2012Metric_Pad1.15x1.40mm_HandSolder, symbol ph_air_shower_controller_hw-rescue:C-Device-ph_main_atsh_hw-rescue-ph_main_atsh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
- removed C37: 4.7uF, Capacitor_Tantalum_SMD:CP_EIA-3216-18_Kemet-A_Pad1.58x1.35mm_HandSolder, symbol ph_air_shower_controller_hw-rescue:CP1-Device-ph_main_atsh_hw-rescue-ph_main_at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
- removed C38: 10nF, Capacitor_SMD:C_0805_2012Metric_Pad1.15x1.40mm_HandSolder, symbol ph_air_shower_controller_hw-rescue:C-Device-ph_main_atsh_hw-rescue-ph_main_atsh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
- removed IR1: HS0038A2, nhantt-kicad-lib:HS0038A2, symbol ph_air_shower_controller_hw-rescue:HS0038A2-ATSH_lib_hw-ph_main_atsh_hw-rescue-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
- removed Q2, Q3, Q5, Q6: LN2302, nhantt-kicad-lib:SOT-23, symbol ph_air_shower_controller_hw-rescue:Q_NMOS_GSD-Device-ph_main_atsh_hw-rescue-ph_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
- removed R23: 0R, Resistor_SMD:R_0805_2012Metric_Pad1.15x1.40mm_HandSolder, symbol ph_air_shower_controller_hw-rescue:R-Device-ph_main_atsh_hw-rescue-ph_main_atsh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
- removed R27, R28, R29, R30, R34, R35, R36, R37, R44, R46: 10k, Resistor_SMD:R_0805_2012Metric_Pad1.15x1.40mm_HandSolder, symbol ph_air_shower_controller_hw-rescue:R-Device-ph_main_atsh_hw-rescue-ph_main_atsh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
- removed R43: 100, Resistor_SMD:R_0805_2012Metric_Pad1.15x1.40mm_HandSolder, symbol ph_air_shower_controller_hw-rescue:R-Device-ph_main_atsh_hw-rescue-ph_main_atsh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
- removed R45: 4.7K, Resistor_SMD:R_0805_2012Metric_Pad1.15x1.40mm_HandSolder, symbol ph_air_shower_controller_hw-rescue:R-Device-ph_main_atsh_hw-rescue-ph_main_atsh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
- removed U5, U6: SM5852, VinhTho_Lib:SM5852, symbol ph_air_shower_controller_hw-rescue:SM5852-ATSH_lib_hw-ph_main_atsh_hw-rescue-ph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
- J4, J7, J8: symbol Connector_Generic:Conn_01x06 -> ph_air_shower_controller_hw-rescue:Conn_01x06-Connector_Generic
Connections:
- net labels removed: I2C1_SCL, I2C1_SDA, I2C2_SCL, I2C2_SDA, IR_rev, SCL1, SCL2, SDA1, SDA2
- wire segments 690 -> 617
- no-connect marks 27 -> 25
