File: ph_air_shower_controller_hw/ph_air_shower_controller_hw.sch (KiCad schematic (older format))
At the start: 199 parts, among them J1 Conn_01x02, J2 Conn_01x02, J3 Conn_01x04, J4 Conn_01x06, J7 Conn_01x06, J8 Conn_01x06, P1 USB_OTG, Q1 C1815, Q4 C1815, Q7 C1815, Q8 LN2302, Q9 LN2302, SW1 RESET, SW2 SW_Push, SW3 SW_Push, SW4 SW_Push, SW5 SW_Push, U1 W25Q80BV, U10 PC817, U11 ULN2803A, U12 PC817, U13 PC817, U14 PC817, U15 PC817, U16 DS18B20, U2 MC34063, U3 MAX485, U4 ASM1117, U7 STM32F103RD, U8 74HC245, U9 PC817, Y1 8Mhz, Y2 32768Khz

Commit message: Updating
Parts:
- removed C1, C2, C40, C41, C42, C43, C44, C46, C48, C49: 100nF, Capacitor_SMD:C_0805_2012Metric_Pad1.15x1.40mm_HandSolder, symbol ph_air_shower_controller_hw-rescue:C-Device-ph_main_atsh_hw-rescue-ph_main_atsh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
- removed C47: 4.7uF, Capacitor_SMD:C_1206_3216Metric_Pad1.42x1.75mm_HandSolder, symbol ph_air_shower_controller_hw-rescue:C-Device-ph_main_atsh_hw-rescue-ph_main_atsh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
- removed D10, D11, D13, D8, D9, D? (x6): 12, nhantt-kicad-lib:SOD-80, symbol ph_air_shower_controller_hw-rescue:D_Zener_ALT-Device-ph_main_atsh_hw-rescue-ph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
- removed D14: LED_STATUS, LED_SMD:LED_0805_2012Metric_Pad1.15x1.40mm_HandSolder, symbol ph_air_shower_controller_hw-rescue:LED_ALT-Device-ph_main_atsh_hw-rescue-ph_mai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
- removed D? (x5): D_ALT, Diode_SMD:D_SOD-123, symbol ph_air_shower_controller_hw-rescue:D_ALT-Device-ph_main_atsh_hw-rescue-ph_main_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
- removed J1: Conn_01x02, nhantt-kicad-lib:TerminalBlock_WAGO-236_2Stift_R5mm_2pol, symbol ph_air_shower_controller_hw-rescue:Conn_01x02-Connector_Generic-ph_main_atsh_hw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
- removed J4, J7, J8: Conn_01x06, VinhTho_Lib:TerminalBlock_WAGO_2.54mm_6P, symbol ph_air_shower_controller_hw-rescue:Conn_01x06-Connector_Generic-ph_air_shower_c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
- removed J?: Conn_01x08, symbol Connector_Generic_lib:Conn_01x08
- removed Q1: C1815, nhantt-kicad-lib:SOT-23, symbol ph_air_shower_controller_hw-rescue:C1815-nhantt-kicad-lib-ph_mcu_base_board_dat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
- removed Q8, Q9: LN2302, nhantt-kicad-lib:SOT-23, symbol ph_air_shower_controller_hw-rescue:Q_NMOS_GSD-Device-ph_main_atsh_hw-rescue-ph_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
- removed Q? (x6): Q_NMOS_GSD, vinhtho_lib:TO-252-2, symbol ph_air_shower_controller_hw-rescue:Q_NMOS_GSD-Device-ph_main_atsh_hw-rescue-ph_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
- removed R10, R4, R6, R7: 100R, Resistor_SMD:R_0805_2012Metric_Pad1.15x1.40mm_HandSolder, symbol ph_air_shower_controller_hw-rescue:R-Device-ph_main_atsh_hw-rescue-ph_main_atsh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
- removed R12, R17: 2.2k, Resistor_SMD:R_0805_2012Metric_Pad1.15x1.40mm_HandSolder, symbol ph_air_shower_controller_hw-rescue:R-Device-ph_main_atsh_hw-rescue-ph_main_atsh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
- removed R13, R2, R3, R50, R52, R54, R58, R61, R? (x17): 10k, Resistor_SMD:R_0805_2012Metric_Pad1.15x1.40mm_HandSolder, symbol ph_air_shower_controller_hw-rescue:R-Device-ph_main_atsh_hw-rescue-ph_main_atsh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
- removed R14, R15, R16: 220, Resistor_SMD:R_0805_2012Metric_Pad1.15x1.40mm_HandSolder, symbol ph_air_shower_controller_hw-rescue:R-Device-ph_main_atsh_hw-rescue-ph_main_atsh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
- removed R18, R5: 20k, Resistor_SMD:R_0805_2012Metric_Pad1.15x1.40mm_HandSolder, symbol ph_air_shower_controller_hw-rescue:R-Device-ph_main_atsh_hw-rescue-ph_main_atsh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
- removed R49, R51, R53, R57: 470, Resistor_SMD:R_0805_2012Metric_Pad1.15x1.40mm_HandSolder, symbol ph_air_shower_controller_hw-rescue:R-Device-ph_main_atsh_hw-rescue-ph_main_atsh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
- removed R59: 0R, Resistor_SMD:R_0805_2012Metric_Pad1.15x1.40mm_HandSolder, symbol ph_air_shower_controller_hw-rescue:R-Device-ph_main_atsh_hw-rescue-ph_main_atsh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
- removed R60: 470k, Resistor_SMD:R_0805_2012Metric_Pad1.15x1.40mm_HandSolder, symbol ph_air_shower_controller_hw-rescue:R-Device-ph_main_atsh_hw-rescue-ph_main_atsh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
- removed R62: 330R, Resistor_SMD:R_0805_2012Metric_Pad1.15x1.40mm_HandSolder, symbol ph_air_shower_controller_hw-rescue:R-Device-ph_main_atsh_hw-rescue-ph_main_atsh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
- removed R63, R8: 4.7k, Resistor_SMD:R_0805_2012Metric_Pad1.15x1.40mm_HandSolder, symbol ph_air_shower_controller_hw-rescue:R-Device-ph_main_atsh_hw-rescue-ph_main_atsh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
- removed R? (x6): 1k, Resistor_SMD:R_0805_2012Metric_Pad1.15x1.40mm_HandSolder, symbol ph_air_shower_controller_hw-rescue:R-Device-ph_main_atsh_hw-rescue-ph_main_atsh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
- removed R? (x5): 10R, Resistor_SMD:R_0805_2012Metric_Pad1.15x1.40mm_HandSolder, symbol ph_air_shower_controller_hw-rescue:R-Device-ph_main_atsh_hw-rescue-ph_main_atsh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
- removed RN1, RN2: 10k, Resistor_SMD:R_Array_Convex_4x0603, symbol ph_air_shower_controller_hw-rescue:R_Pack04-Device-ph_main_atsh_hw-rescue-ph_ma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
- removed SW1: RESET, nhantt-kicad-lib:Button_SW_2PIN, symbol ph_air_shower_controller_hw-rescue:SW_Push-nhantt-kicad-lib-ph_mcu_base_board_d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
- removed U1: W25Q80BV, nhantt-kicad-lib:SOIC-8_3.9x4.9mm_Pitch1.27mm, symbol ph_air_shower_controller_hw-rescue:W25Q80BV-ATSH_lib_hw-ph_main_atsh_hw-rescue-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
- removed U10, U12, U13, U15: PC817, nhantt-kicad-lib:Optocoupler_SMD, symbol mcu_water_sample_hw-rescue:PC817
- removed U11: ULN2803A, nhantt-kicad-lib:SOIC-18W_7.5x11.6mm_Pitch1.27mm, symbol ph_air_shower_controller_hw-rescue:mcu_water_sample_hw-rescue_ULN2803A-mcu_wate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
- removed U16: DS18B20, Package_TO_SOT_THT:TO-92_Inline_Horizontal2, symbol ph_kicad_lib:DS18B20
- removed U3: MAX485, nhantt-kicad-lib:SOIC-8_3.9x4.9mm_Pitch1.27mm, symbol mcu_water_sample_hw-rescue:MAX485-RESCUE-mcu_water_sample_hw
- removed U7: STM32F103RD, nhantt-kicad-lib:LQFP-64_10x10mm_Pitch0.5mm, symbol ph_air_shower_controller_hw-rescue:STM32F103RD-nhantt-kicad-lib-ph_mcu_base_boa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
- removed U?: WT588D, symbol vinhtho_lib:WT588D
- added C? (x5): 100nF, Capacitor_SMD:C_0805_2012Metric_Pad1.15x1.40mm_HandSolder, symbol ph_air_shower_controller_hw-rescue:C-Device-ph_main_atsh_hw-rescue-ph_main_atsh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
- added C? (x2): CP, symbol Device:CP
- added C? (x2): 10uF, Capacitor_SMD:C_0805_2012Metric_Pad1.15x1.40mm_HandSolder, symbol ph_air_shower_controller_hw-rescue:C-Device-ph_main_atsh_hw-rescue-ph_main_atsh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
- added D? (x2): 3V3, symbol Device:D_Zener
- added D? (x2): Bridge_Diode, st-kicad-lib:DB107S, symbol tho_lib:Bridge_Diode
- added D? (x3): D_ALT, Diode_SMD:D_SOD-123, symbol ph_air_shower_controller_hw-rescue:D_ALT-Device-ph_main_atsh_hw-rescue-ph_main_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
- added D?: 5.1, nhantt-kicad-lib:SOD-80, symbol ph_air_shower_controller_hw-rescue:D_Zener_ALT-Device-ph_main_atsh_hw-rescue-ph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
- added J? (x9): Conn_01x02, symbol Connector_Generic:Conn_01x02
- added J?: Conn_01x08, symbol Connector_Generic:Conn_01x08
- added J? (x3): Conn_01x03, symbol Connector_Generic:Conn_01x03
- added Q? (x4): C1815_SOT23, ph_kicad_lib:SOT-23, symbol ph_kicad_lib:C1815_SOT23
- added Q? (x4): Q_NMOS_GSD, vinhtho_lib:TO-252-2, symbol ph_air_shower_controller_hw-rescue:Q_NMOS_GSD-Device-ph_main_atsh_hw-rescue-ph_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
- added R? (x2): 50k, Resistor_SMD:R_0805_2012Metric_Pad1.15x1.40mm_HandSolder, symbol ph_air_shower_controller_hw-rescue:R-Device-ph_main_atsh_hw-rescue-ph_main_atsh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
- added R? (x2): R, Resistor_SMD:R_0805_2012Metric_Pad1.15x1.40mm_HandSolder, symbol ph_air_shower_controller_hw-rescue:R-Device-ph_main_atsh_hw-rescue-ph_main_atsh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
- added R? (x8): 2.2k, Resistor_SMD:R_0805_2012Metric_Pad1.15x1.40mm_HandSolder, symbol ph_air_shower_controller_hw-rescue:R-Device-ph_main_atsh_hw-rescue-ph_main_atsh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
- added R? (x8): 10k, Resistor_SMD:R_0805_2012Metric_Pad1.15x1.40mm_HandSolder, symbol ph_air_shower_controller_hw-rescue:R-Device-ph_main_atsh_hw-rescue-ph_main_atsh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
- added R? (x8): R, symbol Device:R
- added R? (x3): 10R, Resistor_SMD:R_0805_2012Metric_Pad1.15x1.40mm_HandSolder, symbol ph_air_shower_controller_hw-rescue:R-Device-ph_main_atsh_hw-rescue-ph_main_atsh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
- added R? (x3): 470, Resistor_SMD:R_0805_2012Metric_Pad1.15x1.40mm_HandSolder, symbol ph_air_shower_controller_hw-rescue:R-Device-ph_main_atsh_hw-rescue-ph_main_atsh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
- added R? (x2): 10K, Resistor_SMD:R_0805_2012Metric_Pad1.15x1.40mm_HandSolder, symbol ph_air_shower_controller_hw-rescue:R-Device-ph_main_atsh_hw-rescue-ph_main_atsh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
- added SW?: Button_TL3342_5.2x5.2, ph_kicad_lib:BUTTON_TL3342, symbol ph_kicad_lib:Button_TL3342_5.2x5.2
- added U? (x2): INA139, TO_SOT_Packages_SMD:SOT-23-5, symbol tho_lib:INA139
- added U? (x2): PC817, Package_DIP:DIP-4_W7.62mm, symbol Isolator:PC817
- added U? (x3): PC817, nhantt-kicad-lib:Optocoupler_SMD, symbol mcu_water_sample_hw-rescue:PC817
- added U?: STM32F103CxT6, ph_kicad_lib:LQFP-48_7x7mm_Pitch0.5mm, symbol ph_kicad_lib:STM32F103CxT6
- C10: value 100uF -> 220uF
- D12: value 12 -> 5.1
- R19: value 1k -> 1k/1%
- R9: value 3k -> 1k/1%
Connections:
- net labels added: +12V, AIR_DET, CURR1, CURR2, DOOR1, DOOR2, D_SS1, D_SS2, EXIT, EXT2, LAMP_DET, P_SS, RELAY1, RELAY2
- net labels removed: +24V, 485_RX, 485_TX, A, B, CTRL3, CTRL4, CTRL5, CTRL6, DS18B20, IN1, IN2, IN3, IN4, IN5, IN6, OUT1, OUT2, OUT3, OUT4, OUT5, OUT6, PB2, PB3, PB4, PB5, PC6, PC7, SPI2_CLK, SPI2_CS, SPI2_MISO, SPI2_MOSI, UART2_RX, UART2_TX, input1, input2, input3, input4, input5, input6
- wire segments 736 -> 576
- no-connect marks 27 -> 17
Other:
- note removed: "EFROM Data"
- note removed: "Max485\n"
- moved on the sheet: C16, C18, C19, C20, C21, C22, C23, C24, C45, D12, D?, J3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

Commit message: Update Board Relay
Parts:
- removed BT1: Battery_Cell, nhantt-kicad-lib:BT3V3, symbol ph_air_shower_controller_hw-rescue:Battery_Cell-Device-ph_main_atsh_hw-rescue-p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
- removed C10: 220uF, Capacitor_SMD:CP_Elec_8x10.5, symbol ph_air_shower_controller_hw-rescue:CP1-Device-ph_main_atsh_hw-rescue-ph_main_at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
- removed C11, C13, C14, C16, C20, C21, C22, C23, C24, C25, C28, C30, C33, C34, C35, C36, C4, C45, C7, C8, C? (x5): 100nF, Capacitor_SMD:C_0805_2012Metric_Pad1.15x1.40mm_HandSolder, symbol ph_air_shower_controller_hw-rescue:C-Device-ph_main_atsh_hw-rescue-ph_main_atsh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
- removed C12, C19, C5: 10uF, Capacitor_SMD:C_1206_3216Metric_Pad1.42x1.75mm_HandSolder, symbol ph_air_shower_controller_hw-rescue:C-Device-ph_main_atsh_hw-rescue-ph_main_atsh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
- removed C18: 1uF, Capacitor_SMD:C_0805_2012Metric_Pad1.15x1.40mm_HandSolder, symbol ph_air_shower_controller_hw-rescue:C-Device-ph_main_atsh_hw-rescue-ph_main_atsh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
- removed C26, C27: 20pF, Capacitor_SMD:C_0805_2012Metric_Pad1.15x1.40mm_HandSolder, symbol ph_air_shower_controller_hw-rescue:C-Device-ph_main_atsh_hw-rescue-ph_main_atsh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
- removed C3: 100uF, Capacitor_SMD:CP_Elec_8x10.5, symbol ph_air_shower_controller_hw-rescue:CP1-Device-ph_main_atsh_hw-rescue-ph_main_at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
- removed C31, C32: 10pF, Capacitor_SMD:C_0805_2012Metric_Pad1.15x1.40mm_HandSolder, symbol ph_air_shower_controller_hw-rescue:C-Device-ph_main_atsh_hw-rescue-ph_main_atsh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
- removed C6: 47uF, Capacitor_SMD:CP_Elec_5x5.4, symbol ph_air_shower_controller_hw-rescue:CP1-Device-ph_main_atsh_hw-rescue-ph_main_at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
- removed C9: 33pF, Capacitor_SMD:C_0805_2012Metric_Pad1.15x1.40mm_HandSolder, symbol ph_air_shower_controller_hw-rescue:C-Device-ph_main_atsh_hw-rescue-ph_main_atsh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
- removed C? (x2): CP, symbol Device:CP
- removed C? (x2): 10uF, Capacitor_SMD:C_0805_2012Metric_Pad1.15x1.40mm_HandSolder, symbol ph_air_shower_controller_hw-rescue:C-Device-ph_main_atsh_hw-rescue-ph_main_atsh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
- removed D1: D_ALT, Diode_SMD:D_SMB_Handsoldering, symbol ph_air_shower_controller_hw-rescue:D_ALT-Device-ph_main_atsh_hw-rescue-ph_main_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
- removed D12, D?: 5.1, nhantt-kicad-lib:SOD-80, symbol ph_air_shower_controller_hw-rescue:D_Zener_ALT-Device-ph_main_atsh_hw-rescue-ph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
- removed D2: D_TVS_ALT, nhantt-kicad-lib:D_SMA_Standard, symbol ph_air_shower_controller_hw-rescue:D_TVS_ALT-Device-ph_main_atsh_hw-rescue-ph_m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
- removed D3: LED, LED_SMD:LED_0805_2012Metric_Pad1.15x1.40mm_HandSolder, symbol ph_air_shower_controller_hw-rescue:LED-Device-ph_main_atsh_hw-rescue-ph_main_at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
- removed D4: D_Schottky, ph_kicad_lib:D_SMA_Handsoldering, symbol ph_air_shower_controller_hw-rescue:D_Schottky-Device-ph_main_atsh_hw-rescue-ph_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
- removed D5, D? (x4): D_ALT, Diode_SMD:D_SOD-123, symbol ph_air_shower_controller_hw-rescue:D_ALT-Device-ph_main_atsh_hw-rescue-ph_main_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
- removed D6: LED_STATUS, LED_SMD:LED_0805_2012Metric_Pad1.15x1.40mm_HandSolder, symbol ph_air_shower_controller_hw-rescue:LED_ALT-Device-ph_main_atsh_hw-rescue-ph_mai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
- removed D7: DIODE, Diode_SMD:D_SOD-123, symbol ph_air_shower_controller_hw-rescue:DIODE-Simulation_SPICE-ph_main_atsh_hw-rescu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
- removed D? (x2): 3V3, symbol Device:D_Zener
- removed D? (x2): Bridge_Diode, st-kicad-lib:DB107S, symbol tho_lib:Bridge_Diode
- removed F1: Fuse, nhantt-kicad-lib:Fuse_SMD1812, symbol ph_air_shower_controller_hw-rescue:Fuse-Device-ph_main_atsh_hw-rescue-ph_main_a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
- removed J2: Conn_01x02, nhantt-kicad-lib:TerminalBlock_WAGO-236_2Stift_R5mm_2pol, symbol ph_air_shower_controller_hw-rescue:Conn_01x02-Connector_Generic-ph_main_atsh_hw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
- removed J3: Conn_01x04, nhantt-kicad-lib:Pin_Header_Straight_1x04_Pitch2.54mm, symbol mcu_water_sample_hw-rescue:Conn_01x04
- removed J? (x9): Conn_01x02, symbol Connector_Generic:Conn_01x02
- removed J?: Conn_01x08, symbol Connector_Generic:Conn_01x08
- removed J? (x3): Conn_01x03, symbol Connector_Generic:Conn_01x03
- removed L1: L, nhantt-kicad-lib:Inductor_5.2x5.8x4.5, symbol ph_air_shower_controller_hw-rescue:L-Device-ph_main_atsh_hw-rescue-ph_main_atsh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
- removed L2: 30R, Inductor_SMD:L_0805_2012Metric_Pad1.15x1.40mm_HandSolder, symbol ph_air_shower_controller_hw-rescue:L_Small-Device-ph_main_atsh_hw-rescue-ph_mai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
- removed LCD1: ST7920, VinhTho_Lib:ST7920, symbol ph_air_shower_controller_hw-rescue:ST7920-ATSH_lib_hw-ph_main_atsh_hw-rescue-ph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
- removed LS1: Speaker, Buzzer_Beeper:Buzzer_15x7.5RM7.6, symbol ph_air_shower_controller_hw-rescue:mcu_water_sample_hw-rescue_Speaker-mcu_water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
- removed P1: USB_OTG, nhantt-kicad-lib:USB_Micro-B, symbol ph_air_shower_controller_hw-rescue:USB_OTG-RESCUE-esp32bb-nhantt-kicad-lib-ph_m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
- removed Q4, Q7: C1815, nhantt-kicad-lib:SOT-23, symbol ph_air_shower_controller_hw-rescue:C1815-nhantt-kicad-lib-ph_mcu_base_board_dat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
- removed Q? (x4): C1815_SOT23, ph_kicad_lib:SOT-23, symbol ph_kicad_lib:C1815_SOT23
- removed Q? (x4): Q_NMOS_GSD, vinhtho_lib:TO-252-2, symbol ph_air_shower_controller_hw-rescue:Q_NMOS_GSD-Device-ph_main_atsh_hw-rescue-ph_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
- removed R1: 0.15, Resistor_SMD:R_1206_3216Metric_Pad1.42x1.75mm_HandSolder, symbol ph_air_shower_controller_hw-rescue:R-Device-ph_main_atsh_hw-rescue-ph_main_atsh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
- removed R11, R33: 1k, Resistor_SMD:R_0805_2012Metric_Pad1.15x1.40mm_HandSolder, symbol ph_air_shower_controller_hw-rescue:R-Device-ph_main_atsh_hw-rescue-ph_main_atsh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
- removed R19, R9: 1k/1%, Resistor_SMD:R_0805_2012Metric_Pad1.15x1.40mm_HandSolder, symbol ph_air_shower_controller_hw-rescue:R-Device-ph_main_atsh_hw-rescue-ph_main_atsh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
- removed R20, R21: 22R, Resistor_SMD:R_0805_2012Metric_Pad1.15x1.40mm_HandSolder, symbol ph_air_shower_controller_hw-rescue:R-Device-ph_main_atsh_hw-rescue-ph_main_atsh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
- removed R22: 1.5k, Resistor_SMD:R_0805_2012Metric_Pad1.15x1.40mm_HandSolder, symbol ph_air_shower_controller_hw-rescue:R-Device-ph_main_atsh_hw-rescue-ph_main_atsh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
- removed R24, R26, R32, R39, R40, R41, R42, R48, R56, R? (x9): 10k, Resistor_SMD:R_0805_2012Metric_Pad1.15x1.40mm_HandSolder, symbol ph_air_shower_controller_hw-rescue:R-Device-ph_main_atsh_hw-rescue-ph_main_atsh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
- removed R25: 220R, Resistor_SMD:R_0805_2012Metric_Pad1.15x1.40mm_HandSolder, symbol ph_air_shower_controller_hw-rescue:R-Device-ph_main_atsh_hw-rescue-ph_main_atsh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
- removed R31, R38, R? (x8): 2.2k, Resistor_SMD:R_0805_2012Metric_Pad1.15x1.40mm_HandSolder, symbol ph_air_shower_controller_hw-rescue:R-Device-ph_main_atsh_hw-rescue-ph_main_atsh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
- removed R47, R55, R? (x3): 470, Resistor_SMD:R_0805_2012Metric_Pad1.15x1.40mm_HandSolder, symbol ph_air_shower_controller_hw-rescue:R-Device-ph_main_atsh_hw-rescue-ph_main_atsh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
- removed R? (x4): 10R, Resistor_SMD:R_0805_2012Metric_Pad1.15x1.40mm_HandSolder, symbol ph_air_shower_controller_hw-rescue:R-Device-ph_main_atsh_hw-rescue-ph_main_atsh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
- removed R? (x2): 50k, Resistor_SMD:R_0805_2012Metric_Pad1.15x1.40mm_HandSolder, symbol ph_air_shower_controller_hw-rescue:R-Device-ph_main_atsh_hw-rescue-ph_main_atsh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
- removed R? (x2): R, Resistor_SMD:R_0805_2012Metric_Pad1.15x1.40mm_HandSolder, symbol ph_air_shower_controller_hw-rescue:R-Device-ph_main_atsh_hw-rescue-ph_main_atsh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
- removed R? (x8): R, symbol Device:R
- removed R? (x2): 10K, Resistor_SMD:R_0805_2012Metric_Pad1.15x1.40mm_HandSolder, symbol ph_air_shower_controller_hw-rescue:R-Device-ph_main_atsh_hw-rescue-ph_main_atsh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
- removed RV1: R_POT, nhantt-kicad-lib:VR1, symbol ph_air_shower_controller_hw-rescue:R_POT-Device-ph_main_atsh_hw-rescue-ph_main_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
- removed SW2, SW3, SW4, SW5: SW_Push, Button_Switch_THT:SW_PUSH-12mm, symbol ph_air_shower_controller_hw-rescue:SW_Push-nhantt-kicad-lib-ph_mcu_base_board_d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
- removed SW?: Button_TL3342_5.2x5.2, ph_kicad_lib:BUTTON_TL3342, symbol ph_kicad_lib:Button_TL3342_5.2x5.2
- removed U14, U9, U? (x3): PC817, nhantt-kicad-lib:Optocoupler_SMD, symbol mcu_water_sample_hw-rescue:PC817
- removed U2: MC34063, nhantt-kicad-lib:SOIC-8_3.9x4.9mm_Pitch1.27mm, symbol ph_air_shower_controller_hw-rescue:MC34063-nhantt-kicad-lib-motor_driver_water_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
- removed U4: ASM1117, nhantt-kicad-lib:SOT-223, symbol ph_air_shower_controller_hw-rescue:ASM1117-nhantt-kicad-lib-ph_mcu_base_board_d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
- removed U8: 74HC245, nhantt-kicad-lib:TSSOP-20_4.4x6.5mm_Pitch0.65mm, symbol ph_air_shower_controller_hw-rescue:74HC245-ATSH_lib_hw-ph_main_atsh_hw-rescue-p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
- removed U? (x2): INA139, TO_SOT_Packages_SMD:SOT-23-5, symbol tho_lib:INA139
- removed U? (x2): PC817, Package_DIP:DIP-4_W7.62mm, symbol Isolator:PC817
- removed U?: STM32F103CxT6, ph_kicad_lib:LQFP-48_7x7mm_Pitch0.5mm, symbol ph_kicad_lib:STM32F103CxT6
- removed Y1: 8Mhz, nhantt-kicad-lib:Crystal_SMD_HC49-SD, symbol ph_air_shower_controller_hw-rescue:Crystal-Device-ph_main_atsh_hw-rescue-ph_mai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
- removed Y2: 32768Khz, nhantt-kicad-lib:Crystal_Round_Horizontal_3mm_smd, symbol ph_air_shower_controller_hw-rescue:Crystal_GND3-Device-ph_main_atsh_hw-rescue-p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
Connections:
- no-connect marks 17 -> 0
Other:
- note removed: "Input Block\n\n"
- note removed: "LCD ST7920"
- note removed: "Output Block"
- note removed: "Power Block\n"

Commit message: Updating PCB Controller
Parts:
- added BT1: Battery_Cell, vinhtho_lib:BT3V3, symbol ph_air_shower_controller_hw-rescue:Battery_Cell-Device-ph_main_atsh_hw-rescue-p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
- added C1, C11, C13, C14, C16, C17, C20, C21, C22, C23, C24, C25, C28, C29, C30, C33, C34, C35, C36, C37, C38, C4, C45, C7, C8: 100nF, Capacitors_SMD:C_0805_2012Metric_Pad1.15x1.40mm_HandSolder, symbol ph_air_shower_controller_hw-rescue:C-Device-ph_main_atsh_hw-rescue-ph_main_atsh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
- added C10: 220uF, Capacitors_SMD:C_Elec_8x10.2, symbol ph_air_shower_controller_hw-rescue:CP1-Device-ph_main_atsh_hw-rescue-ph_main_at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
- added C12, C15, C19, C2, C5: 10uF, Capacitors_SMD:C_1206_3216Metric_Pad1.42x1.75mm_HandSolder, symbol ph_air_shower_controller_hw-rescue:C-Device-ph_main_atsh_hw-rescue-ph_main_atsh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
- added C18: 1uF, Capacitors_SMD:C_0805_2012Metric_Pad1.15x1.40mm_HandSolder, symbol ph_air_shower_controller_hw-rescue:C-Device-ph_main_atsh_hw-rescue-ph_main_atsh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
- added C26, C27: 20pF, Capacitors_SMD:C_0805_2012Metric_Pad1.15x1.40mm_HandSolder, symbol ph_air_shower_controller_hw-rescue:C-Device-ph_main_atsh_hw-rescue-ph_main_atsh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
- added C3: 100uF, Capacitors_SMD:C_Elec_8x10.2, symbol ph_air_shower_controller_hw-rescue:CP1-Device-ph_main_atsh_hw-rescue-ph_main_at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
- added C31, C32: 10pF, Capacitors_SMD:C_0805_2012Metric_Pad1.15x1.40mm_HandSolder, symbol ph_air_shower_controller_hw-rescue:C-Device-ph_main_atsh_hw-rescue-ph_main_atsh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
- added C6: 47uF, Capacitors_SMD:C_Elec_5x5.4, symbol ph_air_shower_controller_hw-rescue:CP1-Device-ph_main_atsh_hw-rescue-ph_main_at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
- added C9: 33pF, Capacitors_SMD:C_0805_2012Metric_Pad1.15x1.40mm_HandSolder, symbol ph_air_shower_controller_hw-rescue:C-Device-ph_main_atsh_hw-rescue-ph_main_atsh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
- added D1: D_ALT, Diode_SMD:D_SMB_Handsoldering, symbol ph_air_shower_controller_hw-rescue:D_ALT-Device-ph_main_atsh_hw-rescue-ph_main_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
- added D10, D9: 3V3, ph_kicad_lib:D_SOD-80, symbol ph_air_shower_controller_hw-rescue:D_Zener-Device
- added D11, D13, D14, D15, D5: D_ALT, Diode_SMD:D_SOD-123, symbol ph_air_shower_controller_hw-rescue:D_ALT-Device-ph_main_atsh_hw-rescue-ph_main_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
- added D12, D8: 5.1, ph_kicad_lib:D_SOD-80, symbol ph_air_shower_controller_hw-rescue:D_Zener_ALT-Device-ph_main_atsh_hw-rescue-ph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
- added D2: D_TVS_ALT, ph_kicad_lib:D_SMA_Handsoldering, symbol ph_air_shower_controller_hw-rescue:D_TVS_ALT-Device-ph_main_atsh_hw-rescue-ph_m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
- added D3: LED, LED_SMD:LED_0805_2012Metric_Pad1.15x1.40mm_HandSolder, symbol ph_air_shower_controller_hw-rescue:LED-Device-ph_main_atsh_hw-rescue-ph_main_at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
- added D4: D_Schottky, ph_kicad_lib:D_SMA_Handsoldering, symbol ph_air_shower_controller_hw-rescue:D_Schottky-Device-ph_main_atsh_hw-rescue-ph_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
- added D6: LED_STATUS, LED_SMD:LED_0805_2012Metric_Pad1.15x1.40mm_HandSolder, symbol ph_air_shower_controller_hw-rescue:LED_ALT-Device-ph_main_atsh_hw-rescue-ph_mai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
- added D7: DIODE, Diode_SMD:D_SOD-123, symbol ph_air_shower_controller_hw-rescue:DIODE-Simulation_SPICE-ph_main_atsh_hw-rescu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
- added F1: Fuse, ph_kicad_lib:Fuse_SMD1812, symbol ph_air_shower_controller_hw-rescue:Fuse-Device-ph_main_atsh_hw-rescue-ph_main_a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
- added J1, J4: Conn_01x02, vinhtho_lib:TerminalBlock_WAGO_2.54mm_2P, symbol ph_air_shower_controller_hw-rescue:Conn_01x02-Connector_Generic
- added J10, J11, J8, J9: Conn_01x02, vinhtho_lib:TerminalBlock_WAGO-236_2Stift_R5mm_2pol, symbol ph_air_shower_controller_hw-rescue:Conn_01x02-Connector_Generic
- added J12: Conn_01x08, vinhtho_lib:Pin_Header_Straight_1x08_Pitch2.54mm, symbol ph_air_shower_controller_hw-rescue:Conn_01x08-Connector_Generic
- added J2: Conn_01x02, vinhtho_lib:TerminalBlock_WAGO-236_2Stift_R5mm_2pol, symbol ph_air_shower_controller_hw-rescue:Conn_01x02-Connector_Generic-ph_main_atsh_hw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
- added J3: Conn_01x04, vinhtho_lib:Pin_Header_Straight_1x04_Pitch2.54mm, symbol mcu_water_sample_hw-rescue:Conn_01x04
- added J5, J6, J7: Conn_01x03, vinhtho_lib:TerminalBlock_WAGO_2.54mm_3P, symbol ph_air_shower_controller_hw-rescue:Conn_01x03-Connector_Generic
- added L1: L, vinhtho_lib:Inductor_5.2x5.8x4.5, symbol ph_air_shower_controller_hw-rescue:L-Device-ph_main_atsh_hw-rescue-ph_main_atsh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
- added L2: 30R, Inductor_SMD:L_0805_2012Metric_Pad1.15x1.40mm_HandSolder, symbol ph_air_shower_controller_hw-rescue:L_Small-Device-ph_main_atsh_hw-rescue-ph_mai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
- added LCD1: ST7920, vinhtho_lib:ST7920, symbol ph_air_shower_controller_hw-rescue:ST7920-ATSH_lib_hw-ph_main_atsh_hw-rescue-ph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
- added LS1: Speaker, Buzzer_Beeper:Buzzer_15x7.5RM7.6, symbol ph_air_shower_controller_hw-rescue:mcu_water_sample_hw-rescue_Speaker-mcu_water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
- added P1: USB_OTG, vinhtho_lib:USB_Micro-B, symbol ph_air_shower_controller_hw-rescue:USB_OTG-RESCUE-esp32bb-nhantt-kicad-lib-ph_m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
- added Q1, Q2, Q6, Q8: C1815, ph_kicad_lib:SOT-23, symbol ph_kicad_lib:C1815_SOT23
- added Q10, Q3, Q5, Q9: Q_NMOS_GSD, vinhtho_lib:TO-252-2, symbol ph_air_shower_controller_hw-rescue:Q_NMOS_GSD-Device-ph_main_atsh_hw-rescue-ph_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
- added Q4, Q7: C1815, ph_kicad_lib:SOT-23, symbol ph_air_shower_controller_hw-rescue:C1815-nhantt-kicad-lib-ph_mcu_base_board_dat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
- added R1: 0.15, Resistor_SMD:R_1206_3216Metric_Pad1.42x1.75mm_HandSolder, symbol ph_air_shower_controller_hw-rescue:R-Device-ph_main_atsh_hw-rescue-ph_main_atsh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
- added R10, R18, R2, R23, R24, R26, R32, R39, R4, R40, R41, R42, R43, R44, R48, R5, R56, R8: 10k, Resistor_SMD:R_0805_2012Metric_Pad1.15x1.40mm_HandSolder, symbol ph_air_shower_controller_hw-rescue:R-Device-ph_main_atsh_hw-rescue-ph_main_atsh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
- added R11, R33: 1k, Resistor_SMD:R_0805_2012Metric_Pad1.15x1.40mm_HandSolder, symbol ph_air_shower_controller_hw-rescue:R-Device-ph_main_atsh_hw-rescue-ph_main_atsh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
- added R12, R13, R14, R15, R31, R34, R35, R36, R37, R38: 2.2k, Resistor_SMD:R_0805_2012Metric_Pad1.15x1.40mm_HandSolder, symbol ph_air_shower_controller_hw-rescue:R-Device-ph_main_atsh_hw-rescue-ph_main_atsh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
- added R16, R17: 50k, Resistor_SMD:R_0805_2012Metric_Pad1.15x1.40mm_HandSolder, symbol ph_air_shower_controller_hw-rescue:R-Device-ph_main_atsh_hw-rescue-ph_main_atsh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
- added R19, R9: 1k/1%, Resistor_SMD:R_0805_2012Metric_Pad1.15x1.40mm_HandSolder, symbol ph_air_shower_controller_hw-rescue:R-Device-ph_main_atsh_hw-rescue-ph_main_atsh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
- added R20, R21: 22R, Resistor_SMD:R_0805_2012Metric_Pad1.15x1.40mm_HandSolder, symbol ph_air_shower_controller_hw-rescue:R-Device-ph_main_atsh_hw-rescue-ph_main_atsh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
- added R22: 1.5k, Resistor_SMD:R_0805_2012Metric_Pad1.15x1.40mm_HandSolder, symbol ph_air_shower_controller_hw-rescue:R-Device-ph_main_atsh_hw-rescue-ph_main_atsh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
- added R25: 220R, Resistor_SMD:R_0805_2012Metric_Pad1.15x1.40mm_HandSolder, symbol ph_air_shower_controller_hw-rescue:R-Device-ph_main_atsh_hw-rescue-ph_main_atsh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
- added R27, R28, R45, R46: 10R, Resistor_SMD:R_0805_2012Metric_Pad1.15x1.40mm_HandSolder, symbol ph_air_shower_controller_hw-rescue:R-Device-ph_main_atsh_hw-rescue-ph_main_atsh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
- added R29, R30: R, Resistor_SMD:R_2512_6332Metric_Pad1.52x3.35mm_HandSolder, symbol ph_air_shower_controller_hw-rescue:R-Device-ph_main_atsh_hw-rescue-ph_main_atsh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
- added R3, R47, R55, R6, R7: 470, Resistor_SMD:R_0805_2012Metric_Pad1.15x1.40mm_HandSolder, symbol ph_air_shower_controller_hw-rescue:R-Device-ph_main_atsh_hw-rescue-ph_main_atsh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
- added R49, R50: 10K, Resistor_SMD:R_0805_2012Metric_Pad1.15x1.40mm_HandSolder, symbol ph_air_shower_controller_hw-rescue:R-Device-ph_main_atsh_hw-rescue-ph_main_atsh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
- added RV1: R_POT, vinhtho_lib:VR1, symbol ph_air_shower_controller_hw-rescue:R_POT-Device-ph_main_atsh_hw-rescue-ph_main_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
- added SW1: Button_TL3342_5.2x5.2, ph_kicad_lib:BUTTON_TL3342, symbol ph_kicad_lib:Button_TL3342_5.2x5.2
- added SW2, SW3, SW4, SW5: SW_Push, Button_Switch_THT:SW_PUSH-12mm, symbol ph_air_shower_controller_hw-rescue:SW_Push-nhantt-kicad-lib-ph_mcu_base_board_d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
- added U1, U14, U3, U5, U9: PC817, vinhtho_lib:Optocoupler_SMD, symbol mcu_water_sample_hw-rescue:PC817
- added U10: STM32F103CxT6, ph_kicad_lib:LQFP-48_7x7mm_Pitch0.5mm, symbol ph_kicad_lib:STM32F103CxT6
- added U2: MC34063, vinhtho_lib:SOIC-8_3.9x4.9mm_Pitch1.27mm, symbol ph_air_shower_controller_hw-rescue:MC34063-nhantt-kicad-lib-motor_driver_water_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
- added U4: ASM1117, vinhtho_lib:SOT-223, symbol ph_air_shower_controller_hw-rescue:ASM1117-nhantt-kicad-lib-ph_mcu_base_board_d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
- added U6, U7: INA139, Package_TO_SOT_SMD:SOT-23-5, symbol ph_air_shower_controller_hw-rescue:INA139-tho_lib
- added U8: 74HC245, vinhtho_lib:TSSOP-20_4.4x6.5mm_Pitch0.65mm, symbol ph_air_shower_controller_hw-rescue:74HC245-ATSH_lib_hw-ph_main_atsh_hw-rescue-p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
- added Y1: 8Mhz, vinhtho_lib:Crystal_SMD_HC49-SD, symbol ph_air_shower_controller_hw-rescue:Crystal-Device-ph_main_atsh_hw-rescue-ph_mai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
- added Y2: 32768Khz, vinhtho_lib:Crystal_Round_Horizontal_3mm_smd, symbol ph_air_shower_controller_hw-rescue:Crystal_GND3-Device-ph_main_atsh_hw-rescue-p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
Connections:
- new net: BT1.1 (+), C30.1, U10.1 (VBAT)
- new net: D5.2 (A), P1.1 (VCC)
- new net: P1.2 (D-), R20.2
- new net: P1.3 (D+), R21.2, R22.2
- new net: R47.2, U9.1
- new net: J5.2 (Pin_2), R2.2, R47.1
- new net: D6.2 (A), R33.2
- new net: R1.2, U2.1 (Sw_Coll), U2.7 (I_Sense), U2.8 (Drv_Coll)
- new net: D4.1 (K), L1.1, U2.2 (Sw_Emit)
- new net: C9.1, U2.3 (Tim_Cap)
- new net: R19.1, R9.2, U2.5 (V_Sense)
- new net: D3.2 (A), R11.2
- new net: D1.2 (A), D2.2 (A2), F1.1
- new net: D11.1 (K), J10.1 (Pin_1), J8.1 (Pin_1), R29.2, U6.4 (-IN)
- new net: D11.2 (A), J10.2 (Pin_2), J8.2 (Pin_2), Q3.3 (D)
- new net: Q1.3 (C), R18.2, R27.2
- new net: Q3.1 (G), R27.1
- new net: R55.2, U14.1
- new net: D12.2 (A), R55.1
- new net: D12.1 (K), J1.2 (Pin_2)
- new net: D7.1 (A), LS1.2, Q7.3 (C)
- new net: Q7.1 (B), R38.2
- new net: LCD1.15 (PSB), R24.2
- new net: LCD1.20 (BLK), R25.1
- new net: LCD1.3 (Vo), RV1.2
- new net: Q4.1 (B), R31.2
- new net: Q4.3 (C), R25.2
- new net: Q1.1 (B), R14.1
- new net: D13.1 (K), J11.1 (Pin_1), J9.1 (Pin_1), R30.2, U7.4 (-IN)
- new net: D13.2 (A), J11.2 (Pin_2), J9.2 (Pin_2), Q5.3 (D)
- new net: Q2.3 (C), R23.2, R28.2
- new net: Q5.1 (G), R28.1
- new net: Q2.1 (B), R15.1
- new net: R6.2, U3.1
- new net: J6.2 (Pin_2), R5.2, R6.1
- new net: R7.1, U5.1
- new net: J7.2 (Pin_2), R7.2
- new net: D8.1 (K), J4.2 (Pin_2)
- new net: R3.2, U1.1
- new net: D8.2 (A), R3.1
- new net: Q8.3 (C), R44.2, R46.2
- new net: Q10.1 (G), R46.1
- new net: Q8.1 (B), R37.1
- new net: Q6.3 (C), R43.2, R45.2
- new net: Q9.1 (G), R45.1
- new net: Q6.1 (B), R36.1
- new net +12V: C3.1, C4.1, D1.1 (K), D14.1 (K), D15.1 (K), J1.1 (Pin_1), J12.1 (Pin_1), J12.3 (Pin_3), J4.1 (Pin_1), J5.1 (Pin_1), J6.1 (Pin_1), J7.1 (Pin_1), R1.1, R18.1, R2.1, R23.1, R29.1, R30.1, R43.1, R44.1, R5.1, U2.6 (VCC), U6.3 (+IN), U7.3 (+IN)
- new net +3V3: C15.1, C16.1, C19.1, C2.1, C20.1, C21.1, C22.1, C23.1, C37.1, C38.1, C6.1, C7.1, J3.1 (Pin_1), L2.1, R10.1, R12.2, R13.2, R26.1, R33.1, R34.2, R35.2, R39.1, R4.1, R40.1, R41.1, R42.1, R48.1, R49.2, R50.2, R56.1, R8.1, U10.24 (VDD), U10.36 (VDD), U10.48 (VDD), U4.2 (OUT), U4.4 (OUT), U6.5 (V+), U7.5 (V+)
- new net +5V: C10.1, C11.1, C12.2, C13.1, C14.2, C28.1, C5.1, C8.1, D5.1 (K), D7.2 (K), L1.2, LCD1.19 (BLA), LCD1.2 (VDD), LS1.1, R11.1, R9.1, RV1.3, U4.3 (IN), U8.1 (DIR), U8.20 (VCC)
- new net AIR_DET: J12.7 (Pin_7), R50.1, U10.13 (USART2_RX/ADC12_IN3/TIM2_CH4/PA3)
- new net BT1: C33.1, R39.2, SW2.2, U10.21 (PB10/I2C2_SCL/USART3_TX)
- new net BT2: C34.1, R40.2, SW3.2, U10.22 (PB11/I2C2_SDA/USART3_RX)
- new net BT3: C35.1, R41.2, SW4.2, U10.25 (PB12/SPI2_NSS/I2C2_SMBA/USART3_CK/TIM1_BKIN)
- new net BT4: C36.1, R42.2, SW5.2, U10.26 (PB13/SPI2_SCK/USART3_CTS/TIM1_CH1N)
- new net Buzzer: R38.1, U10.46 (PB9/TIM4_CH4)
- new net CTRL1: R35.1, R37.2, U10.30 (USART1_TX/TIM1_CH2/PA9)
- new net CTRL2: R34.1, R36.2, U10.31 (USART1_RX/TIM1_CH3/PA10)
- new net CURR1: C29.1, D10.1 (K), R17.1, U10.10 (WKUP/USART2_CTS/ADC12_IN0/TIM2_CH1_ETR/PA0), U7.1 (OUT)
- new net CURR2: C17.1, D9.1 (K), R16.1, U10.11 (USART2_RTS/ADC12_IN1/TIM2_CH2/PA1), U6.1 (OUT)
- new net DOOR1: R13.1, R15.2, U10.27 (PB14/SPI2_MISO/USART3_RTS/TIM1_CH2N)
- new net DOOR2: R12.1, R14.2, U10.28 (PB15/SPI2_MOSI/TIM1_CH3N)
- new net D_SS1: R48.2, U10.40 (PB4/NJTRST), U9.4
- new net D_SS2: R8.2, U10.41 (PB5/I2C1_SMBA), U3.4
- new net EXIT: C45.1, R56.2, U10.43 (PB7/I2C1_SDA/TIM4_CH2), U14.4
- new net EXT2: C1.1, R4.2, U1.4, U10.45 (PB8/TIM4_CH3)
- new net GND: BT1.2 (-), C1.2, C10.2, C11.2, C12.1, C13.2, C14.1, C15.2, C16.2, C17.2, C18.2, C19.2, C2.2, C20.2, C21.2, C22.2, C23.2, C24.1, C25.1, C26.1, C27.2, C28.2, C29.2, C3.2, C30.2, C31.2, C32.1, C33.2, C34.2, C35.2, C36.2, C37.2, C38.2, C4.2, C45.2, C5.2, C6.2, C7.2, C8.2, C9.2, D10.2 (A), D2.1 (A1), D3.1 (K), D4.2 (A), D9.2 (A), J12.6 (Pin_6), J12.8 (Pin_8), J2.1 (Pin_1), J3.2 (Pin_2), J5.3 (Pin_3), J6.3 (Pin_3), J7.3 (Pin_3), LCD1.1 (VSS), P1.5 (GND), P1.6 (shield), Q1.2 (E), Q10.2 (S), Q2.2 (E), Q3.2 (S), Q4.2 (E), Q5.2 (S), Q6.2 (E), Q7.2 (E), Q8.2 (E), Q9.2 (S), R16.2, R17.2, R19.2, R24.1, R32.2, RV1.1, SW1.1, SW2.1, SW3.1, SW4.1, SW5.1, U1.2, U1.3, U10.23 (VSS), U10.35 (VSS), U10.47 (VSS), U10.8 (VSSA), U14.2, U14.3, U2.4 (GND), U3.2, U3.3, U4.1 (GND), U5.2, U5.3, U6.2 (GND), U7.2 (GND), U8.10 (GND), U8.19 (CE), U9.2, U9.3, Y2.3
- new net LAMP_DET: J12.5 (Pin_5), R49.1, U10.12 (USART2_TX/ADC12_IN2/TIM2_CH3/PA2)
- new net LCD_BL: R31.1, U8.14 (B4)
- new net LCD_CLK: LCD1.6 (E), U8.17 (B1)
- new net LCD_CS: LCD1.4 (RS), U8.18 (B0)
- new net LCD_DATA: LCD1.5 (R/~W), U8.16 (B2)
- new net LCD_RST: LCD1.17 (~RST), U8.15 (B3)
- new net OSC32I: C31.1, U10.3 (PC14/OSC32_IN), Y2.2
- new net OSC32O: C32.2, U10.4 (PC15/OSC32_OUT), Y2.1
- new net OSCI: C26.2, U10.5 (PD0/OSC_IN), Y1.2
- new net OSCO: C27.1, U10.6 (PD1/OSC_OUT), Y1.1
- new net P_SS: R10.2, U10.42 (PB6/I2C1_SCL/TIM4_CH1), U5.4
- new net RELAY1: D15.2 (A), J12.2 (Pin_2), Q10.3 (D)
- new net RELAY2: D14.2 (A), J12.4 (Pin_4), Q9.3 (D)
- new net SPI1_CLK: U10.15 (SPI1_SCK/ADC12_IN5/PA5), U8.3 (A1)
- new net SPI1_CS: U10.14 (SPI1_NSS/USART2_CK/ADC12_IN4/PA4), U8.2 (A0)
- new net SPI1_MOSI: U10.17 (SPI1_MOSI/ADC12_IN7/TIM3_CH2/PA7), U8.4 (A2)
- new net ST_BL: U10.29 (USART1_CK/TIM1_CH1/MCO/PA8), U8.6 (A4)
- new net ST_RST: U10.16 (SPI1_MISO/ADC12_IN6/TIM3_CH1/PA6), U8.5 (A3)
- new net SWCLK: J3.4 (Pin_4), U10.37 (JTCK/SWCLK/PA14)
- new net SWDIO: J3.3 (Pin_3), U10.34 (JTMS/SWDIO/PA13)
- new net USB_DIS: R22.1, U10.38 (JTDI/PA15)
- new net USB_DM: R20.1, U10.32 (USART1_CTS/CANRX/USBDM/TIM1_CH4/PA11)
- new net USB_DP: R21.1, U10.33 (USART1_RTS/CANTX/USBDP/TIM1_ETR/PA12)
- new net VDDA: C18.1, C24.2, L2.2, U10.9 (VDDA)
- new net VIN: F1.2, J2.2 (Pin_2)
- new net booto: R32.1, U10.44 (BOOT0)
- new net led_status: D6.1 (K), U10.39 (PB3/JTDO)
- new net reset: C25.2, R26.2, SW1.2, U10.7 (~NRST)
- no-connect marks 0 -> 17
Other:
- note added: "Input Block\n\n"
- note added: "LCD ST7920"
- note added: "Output Block"
- note added: "Power Block\n"

Commit message: Update Diagram system
Parts:
- SW1: footprint ph_kicad_lib:BUTTON_TL3342 -> vinhtho_lib:Button_SW_2PIN
Changed lines of the file:
@@
 F 0 "SW1" H 7320 5008 50  0000 C CNN
 F 1 "Button_TL3342_5.2x5.2" H 7320 5009 50  0001 C CNN
-F 2 "ph_kicad_lib:BUTTON_TL3342" H 7320 5015 50  0001 C CNN
+F 2 "vinhtho_lib:Button_SW_2PIN" H 7320 5015 50  0001 C CNN
 F 3 "" H 7320 5015 50  0001 C CNN
 F 4 "5.2x5.2MM, H=1.5MM, Waterproof Tact Switch" H 7320 4815 50  0001 C CNN "Desc"
