File: ph_air_shower_controller_hw/ph_air_shower_controller_hw.kicad_pcb (KiCad board)
At the start: 2 copper layers, 150 x 100 mm, 156 parts, among them J1 Conn_01x02, J10 Conn_01x02, J11 Conn_01x02, J12 Conn_01x08, J2 Conn_01x02, J3 Conn_01x04, J4 Conn_01x02, J5 Conn_01x03, J6 Conn_01x03, J7 Conn_01x03, J8 Conn_01x02, J9 Conn_01x02, P1 USB_OTG, Q1 C1815, Q10 Q_NMOS_GSD, Q2 C1815, Q3 Q_NMOS_GSD, Q4 C1815, Q5 Q_NMOS_GSD, Q6 C1815, Q7 C1815, Q8 C1815, Q9 Q_NMOS_GSD, SW1 Button_TL3342_5.2x5.2, SW2 SW_Push, SW3 SW_Push, SW4 SW_Push, SW5 SW_Push, U1 PC817, U10 STM32F103CxT6, U14 PC817, U2 MC34063, U3 PC817, U4 ASM1117, U5 PC817, U6 INA139, U7 INA139, U8 74HC245, U9 PC817, Y1 8Mhz, Y2 32768Khz

Commit message: Update Diagram system
Parts:
- C25, D6, R26, R33: moved to B.Cu
- SW1: footprint ph_kicad_lib:BUTTON_TL3342 -> vinhtho_lib:Button_SW_2PIN; moved to B.Cu
- moved R26 150.5 mm to (169.9, 66.0)
- moved R33 150.2 mm to (173.7, 75.8), turned to 180 degrees
- moved C25 145.4 mm to (173.8, 66.0), turned to 180 degrees
- moved SW1 135.1 mm to (171.9, 69.3)
- moved D6 129.3 mm to (169.9, 75.8)
- moved LS1 65.0 mm to (106.2, 124.9), turned to 270 degrees
- moved D7 63.0 mm to (115.1, 124.7), turned to 90 degrees
- moved Q7 62.4 mm to (118.5, 127.3), turned to 0 degrees
- moved R38 58.9 mm to (118.5, 124.0), turned to 180 degrees
- moved D14 29.2 mm to (122.2, 106.3)
- moved D9 28.8 mm to (143.4, 81.6), turned to 0 degrees
- moved R16 28.8 mm to (143.4, 85.9), turned to 0 degrees
- moved C17 28.8 mm to (143.4, 83.9), turned to 0 degrees
- moved C2 28.8 mm to (140.4, 78.6)
- moved C37 28.8 mm to (136.0, 78.6)
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Routing:
- net +3V3: track 89.0 -> 266.9 mm, vias 0 -> 9
- net +12V: track 41.4 -> 186.4 mm, vias 2 -> 0
- net /AIR_DET: track 0.00 -> 99.6 mm, vias 0 -> 1
- net /LAMP_DET: track 0.00 -> 97.0 mm, vias 0 -> 1
- net /DOOR1: track 0.00 -> 57.6 mm, vias 0 -> 2
- net /USB_DM: track 0.00 -> 56.3 mm, vias 0 -> 2
- net /EXIT: track 0.00 -> 54.4 mm, vias 0 -> 2
- net /USB_DP: track 0.00 -> 53.4 mm, vias 0 -> 2
- net /P_SS: track 0.00 -> 52.2 mm, vias 0 -> 2
- net /EXT2: track 0.00 -> 51.3 mm, vias 0 -> 2
- net /D_SS1: track 0.00 -> 50.2 mm, vias 0 -> 2
- net /D_SS2: track 0.00 -> 49.8 mm, vias 0 -> 2
- net /USB_DIS: track 0.00 -> 49.4 mm, vias 0 -> 2
- net /CURR1: track 0.00 -> 46.7 mm, vias 0 -> 2
- net /CTRL2: track 0.00 -> 46.1 mm, vias 0 -> 2
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- added copper zone on B.Cu, net GND
- added copper zone on F.Cu, net GND
Other:
- net class Default: via_dia 0.8 -> 1; via_drill 0.4 -> 0.5
- board text added: "03042020"
- board text added: "PH_AIR_SHOWER_CABINET_hw"
- board text removed: "+24V"
- board text removed: "19022020"
- board text removed: "PH_BIOLOGICAL_SAFETY_CLASS_I_CABINET_hw"
